File: lora_sx1262.kicad_sch (KiCad schematic)
At the start: 5 parts, among them U3 Wio-SX1262

Commit message: Added front artwork and token on the back
Also:
- Tweaked the trace to the antenna to hopefully better match 50ohm impedance
- Tweaked all traces to use fillet on all corners
- Added/fixed parts information

Signed-off-by: Thomas Flummer <tf@flummer.net>
Parts:
- AE1, C5, C9: now left out of the parts list
- U3: value Wio-SX1262 -> Wio-SX1262 / 113991436; Manufacturer SenseCAP -> seeed studio
Changed lines of the file:
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@@
 		(unit 1)
 		(exclude_from_sim no)
-		(in_bom yes)
+		(in_bom no)
 		(on_board yes)
 		(dnp yes)
@@
 			)
 		)
-		(property "Value" "Wio-SX1262"
+		(property "Value" "Wio-SX1262 / 113991436"
 			(at 85.09 68.58 0)
 			(effects
@@
 			)
 		)
-		(property "Datasheet" ""
+		(property "Datasheet" "https://files.seeedstudio.com/products/SenseCAP/Wio_SX1262/Wio-SX1262_Module_Datasheet.pdf"
 			(at 85.09 80.01 0)
 			(effects
@@
 			)
 		)
-		(property "Manufacturer" "SenseCAP"
+		(property "Manufacturer" "seeed studio"
 			(at 85.09 91.44 0)
 			(effects
@@
 		(unit 1)
 		(exclude_from_sim no)
-		(in_bom yes)
+		(in_bom no)
 		(on_board yes)
 		(dnp no)
@@
 		(unit 1)
 		(exclude_from_sim no)
-		(in_bom yes)
+		(in_bom no)
 		(on_board yes)
 		(dnp yes)
